File: Necklace.sch (KiCad schematic (older format))
At the start: 29 parts, among them P1 PICOBLADE_5_HDR_RA, P2 PICOBLADE_5_HDR_RA, SW1 CK_KMR2, U1 ADXL345, U2 MSP430G2452IPW14

Commit message: started layout
Parts:
- removed BATT1: CR2032_SMT_HOLDER_2PIN, SMTU-2032, symbol CR2032_SMT_HOLDER_2PIN
- added BATT1: CR2032_SMT_HOLDER_2pin, Nightmechanic_PCB:SMTU_2032, symbol CR2032_SMT_HOLDER_2pin
- C1, C2, C5, C6: footprint 0805 -> Capacitors_SMD:C_0805
- C3, C4: footprint 1206 -> Capacitors_SMD:C_1206
- D1, D2, D3, D4, D5, D6: footprint SMD_MiniLED -> Nightmechanic_PCB:SMD_MiniLED
- P1, P2: footprint Molex_PICOBLADE_5_HDR_RA -> Connectors_Molex:Connector_Molex_PicoBlade_53261-0571
- R1, R10, R11, R2, R3, R4, R5, R6, R7, R8, R9: footprint 0805 -> Resistors_SMD:R_0805
- SW1: footprint CK_KMR2 -> Nightmechanic_PCB:CK_KMR2
- U1: footprint AD_LGA14 -> (none)
- U2: footprint 14PW -> Nightmechanic_PCB:TI_PW14_TSSOP14
Connections:
- wire segments 91 -> 96
Other:
- moved on the sheet: C3, C5, C6, R4, SW1, U2

Commit message: layout continues
Parts:
- U1: footprint (none) -> Nightmechanic_PCB:AD_LGA14
Changed lines of the file:
@@
 F 0 "U1" H 2000 5850 60  0000 C CNN
 F 1 "ADXL345" H 3100 5850 60  0000 C CNN
-F 2 "" H 2600 4750 40  0001 C CIN
+F 2 "Nightmechanic_PCB:AD_LGA14" H 2600 4750 40  0001 C CIN
 F 3 "http://www.analog.com/static/imported-files/data_sheets/ADXL345.pdf" H 2600 5950 60  0001 C CNN
 	1    2600 5150

Commit message: and some more layout
Changed lines of the file:
@@
 Text Label 5550 1150 0    60   ~ 0
 I2C_SDA
+Text Label 5550 1450 0    60   ~ 0
+ACC_INT1
 Text Label 5550 1350 0    60   ~ 0
-ACC_INT1
-Text Label 5550 1450 0    60   ~ 0
 ACC_INT2
 $Comp

Commit message: late night layout...
Connections:
- wire segments 96 -> 104
Other:
- moved on the sheet: P2, SW1
Changed lines of the file:
@@
 L GND #PWR011
 U 1 1 539E0D8D
-P 1500 7300
-F 0 "#PWR011" H 1500 7300 30  0001 C CNN
-F 1 "GND" H 1500 7230 30  0001 C CNN
-F 2 "" H 1500 7300 60  0000 C CNN
-F 3 "" H 1500 7300 60  0000 C CNN
-	1    1500 7300
+P 1350 7400
+F 0 "#PWR011" H 1350 7400 30  0001 C CNN
+F 1 "GND" H 1350 7330 30  0001 C CNN
+F 2 "" H 1350 7400 60  0000 C CNN
+F 3 "" H 1350 7400 60  0000 C CNN
+	1    1350 7400
 	1    0    0    -1
 $EndComp
@@
 U 1 1 539E1778
 P 6750 2600
-F 0 "P1" H 6750 2850 60  0000 C CNN
-F 1 "PICOBLADE_5_HDR_RA" H 6750 2750 60  0000 C CNN
+F 0 "P1" H 6950 2900 60  0000 C CNN
+F 1 "PICOBLADE_5_HDR_RA" H 7300 2700 60  0000 C CNN
 F 2 "Connectors_Molex:Connector_Molex_PicoBlade_53261-0571" H 6750 2000 40  0000 C CIN
 F 3 "http://www.molex.com/molex/products/datasheet.jsp?part=active/0532610571_PCB_HEADERS.xml" H 6750 2850 60  0001 C CNN
@@
 L PICOBLADE_5_HDR_RA P2
 U 1 1 539E18A5
-P 6750 1050
-F 0 "P2" H 6750 1300 60  0000 C CNN
-F 1 "PICOBLADE_5_HDR_RA" H 6750 1200 60  0000 C CNN
-F 2 "Connectors_Molex:Connector_Molex_PicoBlade_53261-0571" H 6750 450 40  0000 C CIN
-F 3 "http://www.molex.com/molex/products/datasheet.jsp?part=active/0532610571_PCB_HEADERS.xml" H 6750 1300 60  0001 C CNN
-	1    6750 1050
-	1    0    0    -1
-$EndComp
-Text Label 5550 1050 0    60   ~ 0
+P 9000 1300
+F 0 "P2" H 9000 1550 60  0000 C CNN
+F 1 "PICOBLADE_5_HDR_RA" H 9000 1450 60  0000 C CNN
+F 2 "Connectors_Molex:Connector_Molex_PicoBlade_53261-0571" H 9000 700 40  0000 C CIN
+F 3 "http://www.molex.com/molex/products/datasheet.jsp?part=active/0532610571_PCB_HEADERS.xml" H 9000 1550 60  0001 C CNN
+	1    9000 1300
+	1    0    0    -1
+$EndComp
+Text Label 7800 1300 0    60   ~ 0
 I2C_SCL
-Text Label 5550 1150 0    60   ~ 0
+Text Label 7800 1400 0    60   ~ 0
 I2C_SDA
-Text Label 5550 1450 0    60   ~ 0
+Text Label 7800 1700 0    60   ~ 0
 ACC_INT1
-Text Label 5550 1350 0    60   ~ 0
+Text Label 7800 1600 0    60   ~ 0
 ACC_INT2
 $Comp
 L GND #PWR018
 U 1 1 539E1A93
-P 5200 1350
-F 0 "#PWR018" H 5200 1350 30  0001 C CNN
-F 1 "GND" H 5200 1280 30  0001 C CNN
-F 2 "" H 5200 1350 60  0000 C CNN
-F 3 "" H 5200 1350 60  0000 C CNN
-	1    5200 1350
+P 7450 1600
+F 0 "#PWR018" H 7450 1600 30  0001 C CNN
+F 1 "GND" H 7450 1530 30  0001 C CNN
+F 2 "" H 7450 1600 60  0000 C CNN
+F 3 "" H 7450 1600 60  0000 C CNN
+	1    7450 1600
 	1    0    0    -1
 $EndComp
@@
 	1450 4900 1450 4700
 Wire Wire Line
-	1500 7250 1500 7300
+	1350 7250 1350 7400
 Wire Wire Line
 	3600 5100 5150 5100
@@
 	6400 3000 5400 3000
 Wire Wire Line
-	6400 1050 5400 1050
-Wire Wire Line
-	6400 1150 5400 1150
-Wire Wire Line
-	5200 1250 6400 1250
-Wire Wire Line
-	6400 1350 5400 1350
-Wire Wire Line
-	6400 1450 5400 1450
-Wire Wire Line
-	5200 1250 5200 1350
+	8650 1300 7650 1300
+Wire Wire Line
+	8650 1400 7650 1400
+Wire Wire Line
+	7450 1500 8650 1500
+Wire Wire Line
+	8650 1600 7650 1600
+Wire Wire Line
+	8650 1700 7650 1700
+Wire Wire Line
+	7450 1500 7450 1600
 Wire Wire Line
 	1250 2050 1250 2150
@@
 L CK_KMR2 SW1
 U 1 1 53A9C6EB
-P 1200 6950
-F 0 "SW1" H 1200 7300 50  0000 C CNN
-F 1 "CK_KMR2" H 1175 6600 50  0000 C CNN
-F 2 "Nightmechanic_PCB:CK_KMR2" H 1175 6500 40  0000 C CIN
-F 3 "http://www.ck-components.com/kmr-2/tactile,10572,en.html" H 1500 7500 60  0001 C CNN
-	1    1200 6950
+P 1050 6950
+F 0 "SW1" H 1050 7300 50  0000 C CNN
+F 1 "CK_KMR2" H 1025 6600 50  0000 C CNN
+F 2 "Nightmechanic_PCB:CK_KMR2" H 1025 6500 40  0000 C CIN
+F 3 "http://www.ck-components.com/kmr-2/tactile,10572,en.html" H 1350 7500 60  0001 C CNN
+	1    1050 6950
 	1    0    0    -1
 $EndComp
@@
 Wire Notes Line
 	3400 1600 3900 1600
-Wire Wire Line
-	1500 6800 1500 6650
-NoConn ~ 900  6650
-NoConn ~ 900  7250
+NoConn ~ 750  7250
 Wire Notes Line
 	3400 1600 3400 1450
@@
 Text Notes 6900 2950 0    60   ~ 0
 External power input / current measurement\n\n\nMCU SBW (programing port)
-Text Notes 6900 1250 0    60   ~ 0
+Text Notes 9150 1500 0    60   ~ 0
 Accelerometer debug connector
 Wire Wire Line
@@
 	1    0    0    -1
 $EndComp
+NoConn ~ 1350 6650
+Wire Wire Line
+	1500 6800 1500 6450
+Wire Wire Line
+	1500 6450 750  6450
+Wire Wire Line
+	750  6450 750  6650
+$Comp
+L GND #PWR?
+U 1 1 54CAB345
+P 9000 2300
+F 0 "#PWR?" H 9000 2300 30  0001 C CNN
+F 1 "GND" H 9000 2230 30  0001 C CNN
+F 2 "" H 9000 2300 60  0000 C CNN
+F 3 "" H 9000 2300 60  0000 C CNN
+	1    9000 2300
+	1    0    0    -1
+$EndComp
+$Comp
+L GND #PWR?
+U 1 1 54CAB359
+P 9250 750
+F 0 "#PWR?" H 9250 750 30  0001 C CNN
+F 1 "GND" H 9250 680 30  0001 C CNN
+F 2 "" H 9250 750 60  0000 C CNN
+F 3 "" H 9250 750 60  0000 C CNN
+	1    9250 750
+	1    0    0    -1
+$EndComp
+Wire Wire Line
+	9250 750  9250 600
+Wire Wire Line
+	9250 600  9000 600
+Wire Wire Line
+	9000 600  9000 750
+$Comp
+L GND #PWR?
+U 1 1 54CAB440
+P 6750 3600
+F 0 "#PWR?" H 6750 3600 30  0001 C CNN
+F 1 "GND" H 6750 3530 30  0001 C CNN
+F 2 "" H 6750 3600 60  0000 C CNN
+F 3 "" H 6750 3600 60  0000 C CNN
+	1    6750 3600
+	1    0    0    -1
+$EndComp
+$Comp
+L GND #PWR?
+U 1 1 54CAB454
+P 7100 2050
+F 0 "#PWR?" H 7100 2050 30  0001 C CNN
+F 1 "GND" H 7100 1980 30  0001 C CNN
+F 2 "" H 7100 2050 60  0000 C CNN
+F 3 "" H 7100 2050 60  0000 C CNN
+	1    7100 2050
+	1    0    0    -1
+$EndComp
+Wire Wire Line
+	7100 2050 7100 1900
+Wire Wire Line
+	7100 1900 6750 1900
+Wire Wire Line
+	6750 1900 6750 2050
 $EndSCHEMATC

Commit message: finished layout, hopeflly
Connections:
- net labels added: ADC_VS, MCU_LED1, MCU_LED2, MCU_LED3, MCU_LED4, MCU_LED5, MCU_LED6, V_BATT
Changed lines of the file:
@@
 	750  6450 750  6650
 $Comp
-L GND #PWR?
+L GND #PWR024
 U 1 1 54CAB345
 P 9000 2300
-F 0 "#PWR?" H 9000 2300 30  0001 C CNN
+F 0 "#PWR024" H 9000 2300 30  0001 C CNN
 F 1 "GND" H 9000 2230 30  0001 C CNN
 F 2 "" H 9000 2300 60  0000 C CNN
@@
 $EndComp
 $Comp
-L GND #PWR?
+L GND #PWR025
 U 1 1 54CAB359
 P 9250 750
-F 0 "#PWR?" H 9250 750 30  0001 C CNN
+F 0 "#PWR025" H 9250 750 30  0001 C CNN
 F 1 "GND" H 9250 680 30  0001 C CNN
 F 2 "" H 9250 750 60  0000 C CNN
@@
 	9000 600  9000 750
 $Comp
-L GND #PWR?
+L GND #PWR026
 U 1 1 54CAB440
 P 6750 3600
-F 0 "#PWR?" H 6750 3600 30  0001 C CNN
+F 0 "#PWR026" H 6750 3600 30  0001 C CNN
 F 1 "GND" H 6750 3530 30  0001 C CNN
 F 2 "" H 6750 3600 60  0000 C CNN
@@
 $EndComp
 $Comp
-L GND #PWR?
+L GND #PWR027
 U 1 1 54CAB454
 P 7100 2050
-F 0 "#PWR?" H 7100 2050 30  0001 C CNN
+F 0 "#PWR027" H 7100 2050 30  0001 C CNN
 F 1 "GND" H 7100 1980 30  0001 C CNN
 F 2 "" H 7100 2050 60  0000 C CNN
@@
 Wire Wire Line
 	6750 1900 6750 2050
+Text Label 1100 4700 0    60   ~ 0
+ADC_VS
+Text Label 8650 4500 0    60   ~ 0
+MCU_LED1
+Text Label 8650 4600 0    60   ~ 0
+MCU_LED2
+Text Label 8650 4700 0    60   ~ 0
+MCU_LED3
+Text Label 8650 4800 0    60   ~ 0
+MCU_LED4
+Text Label 8650 4900 0    60   ~ 0
+MCU_LED5
+Text Label 8650 5000 0    60   ~ 0
+MCU_LED6
+Text Label 1800 800  0    60   ~ 0
+V_BATT
 $EndSCHEMATC
