File: Necklace.kicad_pcb (KiCad board)
At the start: 2 copper layers, 28 parts, among them P1 PICOBLADE_5_HDR_RA, P2 PICOBLADE_5_HDR_RA, SW1 CK_KMR2, U2 MSP430G2452IPW14

Commit message: layout continues
Parts:
- added U1: ADXL345, Nightmechanic_PCB:AD_LGA14, F.Cu at (112.9, 114.0)
- R1: footprint Resistors_SMD:R_0805 -> Resistors_SMD:R_0805_HandSoldering
- U2: footprint Nightmechanic_PCB:TI_PW14_TSSOP14 -> TI_PW14_TSSOP14
- moved R1 15.7 mm to (97.5, 118.2)
- moved P2 13.4 mm to (119.2, 125.8), turned to 270 degrees
- moved P1 13.3 mm to (106.0, 125.3), turned to 90 degrees
- moved C4 9.97 mm to (111.0, 110.1), turned to 0 degrees
- moved C2 8.84 mm to (115.8, 110.1)
- moved R11 8.10 mm to (105.5, 113.5)
- moved R3 6.66 mm to (122.1, 113.8), turned to 270 degrees
- moved R2 6.65 mm to (119.0, 113.8), turned to 270 degrees
- moved C1 4.22 mm to (111.0, 107.4), turned to 0 degrees

Commit message: and some more layout
Parts:
- moved D6 42.5 mm to (115.0, 90.0)
- moved D4 29.5 mm to (120.5, 133.0)
- moved R10 26.0 mm to (121.5, 92.9), turned to 90 degrees
- moved R8 20.4 mm to (126.6, 116.0), turned to 270 degrees
- moved D5 18.5 mm to (126.0, 104.5), turned to 270 degrees
- moved R4 10.9 mm to (119.0, 111.5), turned to 90 degrees
- moved R6 7.49 mm to (101.0, 96.5), turned to 180 degrees
- moved R5 5.95 mm to (102.0, 116.0)
- moved C6 5.73 mm to (107.5, 99.0), turned to 180 degrees
- moved R9 4.13 mm to (119.0, 98.0)
- moved R7 3.15 mm to (103.5, 92.9), turned to 90 degrees
- moved U1 3.08 mm to (112.5, 117.0)
- moved SW1 2.91 mm to (125.5, 117.5)
- moved C4 2.88 mm to (109.5, 112.5)
- moved C2 2.73 mm to (114.5, 112.5)
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Connections:
- P2 pad 4: /ACC_INT1 -> /ACC_INT2
- P2 pad 5: /ACC_INT2 -> /ACC_INT1
Routing:
- net +BATT: track 0.00 -> 69.1 mm, vias 0 -> 5
- net /ACC_INT1: track 0.00 -> 65.0 mm, vias 0 -> 3
- net /SBWTDIO: track 0.00 -> 48.8 mm, vias 0 -> 2
- net Net-(R8-Pad1): track 0.00 -> 37.9 mm, vias 0 -> 2
- net /ACC_INT2: track 0.00 -> 37.4 mm, vias 0 -> 3
- net /I2C_SDA: track 0.00 -> 34.3 mm, vias 0 -> 3
- net /SBWTCK: track 0.00 -> 29.3 mm, vias 0 -> 1
- net Net-(BATT1-Pad2): track 0.00 -> 28.9 mm, vias 0 -> 2
- net Net-(R10-Pad1): track 0.00 -> 27.6 mm
- net /I2C_SCL: track 0.00 -> 23.3 mm, vias 0 -> 2
- net GND: track 0.00 -> 20.0 mm
- net Net-(D4-Pad1): track 0.00 -> 19.0 mm
- net Net-(D1-Pad1): track 0.00 -> 17.8 mm
- net Net-(R7-Pad1): track 0.00 -> 16.5 mm
- net Net-(R6-Pad1): track 0.00 -> 15.8 mm
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Other:
- board outline added: 41 x 56.1 mm
- net class Default: clearance 0.254 -> 0.3; trace_width 0.254 -> 0.3; via_dia 0.889 -> 1; via_drill 0.635 -> 0.6
- rule trace_clearance: 0.254 -> 0.3

Commit message: late night layout...
Parts:
- P1: footprint Connectors_Molex:Connector_Molex_PicoBlade_53261-0571 -> Nightmechanic_PCB:Connector_Molex_PicoBlade_53261-0571
- P2: footprint Connectors_Molex:Connector_Molex_PicoBlade_53261-0571 -> Connector_Molex_PicoBlade_53261-0571
- SW1: footprint Oddities:NetTie-III_SMD -> Nightmechanic_PCB:CK_KMR2
- moved SW1 1.17 mm to (126.3, 116.7)
- moved C1 0.55 mm to (109.5, 109.0)
- moved C4 0.42 mm to (109.5, 112.1)
Connections:
- SW1 pad 1: Net-(SW1-Pad1) -> /SBWTDIO
- SW1 pad 2: /SBWTDIO -> Net-(SW1-Pad2)
Routing:
- net GND: track 20.0 -> 83.0 mm, vias 0 -> 16
- net Net-(C1-Pad1): track 12.8 -> 20.1 mm
- net /SBWTDIO: track 48.8 -> 53.2 mm
- net /ACC_INT1: track 65.0 -> 60.6 mm
- net +BATT: track 69.1 -> 72.9 mm, vias 5 -> 7
- net Net-(R8-Pad1): track 37.9 -> 39.8 mm, vias 2 -> 4
- net /SBWTCK: track 29.3 -> 28.0 mm
- net /I2C_SCL: track 23.3 -> 23.9 mm
- added copper zone on B.Cu, net +BATT
- added copper zone on B.Cu, net GND
- added copper zone on F.Cu, net GND
- added copper zone on F.Cu, net Net-(C1-Pad1)
Other:
- net class Default: clearance 0.3 -> 0.25
- rule trace_clearance: 0.3 -> 0.25
- board text added: "CUT OUT"

Commit message: finished layout, hopeflly
Parts:
- added VAL: REF, Logos:Gears_F.SilkS_8mm, B.Cu at (100.8, 97.2)
- added VAL: REF, Logos:OSHW_F.SilkS_8mm, B.Cu at (124.4, 110.4)
- moved R11 0.06 mm to (105.5, 116.1)
Connections:
- net Net-(BATT1-Pad2) renamed /V_BATT
- net Net-(C1-Pad1) renamed /ADC_VS
- net Net-(R10-Pad1) renamed /MCU_LED1
- net Net-(R5-Pad1) renamed /MCU_LED6
- net Net-(R6-Pad1) renamed /MCU_LED5
- net Net-(R7-Pad1) renamed /MCU_LED4
- net Net-(R8-Pad1) renamed /MCU_LED3
- net Net-(R9-Pad1) renamed /MCU_LED2
Routing:
- net GND: track 83.0 -> 55.8 mm, vias 16 -> 15
- net +BATT: track 72.9 -> 90.6 mm, vias 7 -> 11
- net /ACC_INT1: track 60.6 -> 56.1 mm
- net /MCU_LED5: track 15.8 -> 13.3 mm
- net /MCU_LED4: track 16.5 -> 14.2 mm
- net /MCU_LED6: track 14.5 -> 13.1 mm
- added copper zone on F.Cu, net +BATT
Other:
- board text added: "Gali's Necklace V1.0 © 2015 Nightmechanic"

Commit message: V1.0 ready to fab
Other:
- rule via_min_drill: 0.508 -> 0.4
- rule via_min_size: 0.889 -> 0.8
